Commit message: Änderung in Sick URDF -> Docker kann nicht mit der Variable arbeiten

File: src/sick_scan/urdf/sick_scan.urdf.xacro (robot description, xacro)
@@ -50,5 +50,5 @@
       <visual>
         <geometry>
-          <mesh filename="${mesh}" />
+          <mesh filename="package://sick_scan/meshes/sick_tim_5xx.stl" />
         </geometry>
         <material name="blue" >
@@ -58,5 +58,5 @@
       <collision>
         <geometry>
-          <mesh filename="${mesh}" />
+          <mesh filename="package://sick_scan/meshes/sick_tim_5xx.stl" />
         </geometry>
       </collision>
