Commit message: Physics Parameter verändert + max V

File: src/floribot_simulation/urdf/Floribot_final.urdf.xacro (robot description, xacro)
@@ -49,8 +49,9 @@
   <!-- hardware_interface/VelocityJointInterface -->
   <gazebo reference="${position}">
-    <mu1 value="0.45"/>
-    <mu2 value="0.45"/>
-    <kp value="100000000.0" />
+    <mu1 value="0.5"/>
+    <mu2 value="0.5"/>
+    <kp value="10000000.0" />
     <kd value="1.0" />
+    <fdir1 value="1 0 0"/>
   </gazebo>
 </xacro:macro>
@@ -259,4 +260,5 @@
        <axis xyz="0 1 0"/>
        <origin xyz="${x_joint_wheel_front} ${y_joint_wheel_front} 0"/>
+        <limit effort="1.0" velocity="14.2857" />
   </joint>
 <!-- Transmission -->
@@ -292,4 +294,5 @@
        <axis xyz="0 1 0"/>
        <origin xyz="${x_joint_wheel_front} -${y_joint_wheel_front} 0"/>
+       <limit effort="1.0" velocity="14.2857" />
   </joint>
 <!-- Transmission -->
@@ -325,4 +328,5 @@
        <axis xyz="0 1 0"/>
        <origin xyz="${x_joint_wheel_back} -${y_joint_wheel_back} 0"/>
+       <limit effort="1.0" velocity="14.2857" />
   </joint>
 <!-- Transmission -->
@@ -358,4 +362,5 @@
        <axis xyz="0 1 0"/>
        <origin xyz="${x_joint_wheel_back} ${y_joint_wheel_back} 0"/>
+       <limit effort="1.0" velocity="14.2857" />
   </joint>
 <!-- Transmission -->

Commit message: Add: Kamera Halteurng

File: src/floribot_simulation/urdf/Floribot_final.urdf.xacro (robot description, xacro)
@@ -22,7 +22,7 @@
 <xacro:property name="laser_height" value="0.03" />
 <!-- Kameraparameter -->
-<xacro:property name="x_camera_front" value="0.29" />
-<xacro:property name="x_camera_back" value="-0.315" />
-<xacro:property name="camera_height" value="0.275" />
+<xacro:property name="x_camera_front" value="0.3220" />
+<xacro:property name="x_camera_back" value="-0.347" />
+<xacro:property name="camera_height" value="0.267" />
 <xacro:property name="camera_angle" value="0.26" />
 <!--Verbindungsgelenkparameter (Skizze: |Vorderwagen|I==|Hinterwagen| -> I: Vertikaler Teil, ==: Horizontaler Teil) -->
@@ -104,4 +104,48 @@
     <origin xyz="${x_camera_front} 0 ${camera_height}" rpy="0 ${camera_angle} 0"/>
   </xacro:sensor_d435i>
+  <link name="CameraFrontPositiv">
+      <visual>
+    	  <origin xyz="${len_wagen_vorne/2-0.06} -0.0225 ${height_wagen*2/3+0.033}" rpy="0 1.57 0"/>
+        <axis xyz="0 0 0"/>
+          <geometry>
+              <!-- <box size="${len_wagen_vorne} ${width_wagen} ${height_wagen}"/> -->
+              <mesh filename="package://floribot_simulation/meshes/Anschluss_Item_positiv.stl" scale="0.001 0.001 0.001" />
+          </geometry>
+          <material name="c">
+              <color rgba="0 0.9 0.9 1.0"/>
+          </material>
+      </visual>
+	  <inertial>
+		<mass value="0.1"/>
+        <inertia ixx="0.0" ixy="0.0" ixz="0.0" iyy="0.0" iyz="0.0" izz="0.0"/>
+      </inertial>
+  </link>
+  <joint name="jointCameraFrontPositiv" type="fixed">
+       <parent link="base_link"/>
+       <child link="CameraFrontPositiv"/>
+	   <origin xyz="0 0 0" rpy="0 0 0"/>
+  </joint>
+  <link name="CameraFrontNegativ">
+      <visual>
+    	  <origin xyz="${len_wagen_vorne/2} -0.006 ${height_wagen*2/3+0.0410}" rpy="${-camera_angle-1.57} 0 -1.57"/>
+        <axis xyz="0 0 0"/>
+          <geometry>
+              <!-- <box size="${len_wagen_vorne} ${width_wagen} ${height_wagen}"/> -->
+              <mesh filename="package://floribot_simulation/meshes/Anschluss_Item_negativ.stl" scale="0.001 0.001 0.001" />
+          </geometry>
+          <material name="c">
+              <color rgba="0 0.9 0.9 1.0"/>
+          </material>
+      </visual>
+	  <inertial>
+		<mass value="0.1"/>
+        <inertia ixx="0.0" ixy="0.0" ixz="0.0" iyy="0.0" iyz="0.0" izz="0.0"/>
+      </inertial>
+  </link>
+  <joint name="jointCameraFrontNegativ" type="fixed">
+       <parent link="CameraFrontPositiv"/>
+       <child link="CameraFrontNegativ"/>
+	   <origin xyz="0 0 0" rpy="0 0 0"/>
+  </joint>
   <!-- Laserscanner vorne -->
   <joint name="joint_front_laser" type="fixed">
@@ -247,4 +291,48 @@
     <origin xyz="${x_camera_back} 0 ${camera_height}" rpy="0 ${camera_angle} 3.14"/>
   </xacro:sensor_d435i>
+  <link name="CameraRearPositiv">
+      <visual>
+    	  <origin xyz="${-len_wagen_hinten/2+0.021} +0.0225 ${height_wagen*2/3+0.033}" rpy="0 1.57 3.141"/>
+        <axis xyz="0 0 0"/>
+          <geometry>
+              <!-- <box size="${len_wagen_vorne} ${width_wagen} ${height_wagen}"/> -->
+              <mesh filename="package://floribot_simulation/meshes/Anschluss_Item_positiv.stl" scale="0.001 0.001 0.001" />
+          </geometry>
+          <material name="c">
+              <color rgba="0 0.9 0.9 1.0"/>
+          </material>
+      </visual>
+	  <inertial>
+		<mass value="0.1"/>
+        <inertia ixx="0.0" ixy="0.0" ixz="0.0" iyy="0.0" iyz="0.0" izz="0.0"/>
+      </inertial>
+  </link>
+  <joint name="jointCameraRearPositiv" type="fixed">
+       <parent link="Hinterwagen"/>
+       <child link="CameraRearPositiv"/>
+	   <origin xyz="0 0 0" rpy="0 0 0"/>
+  </joint>
+  <link name="CameraRearNegativ">
+      <visual>
+    	  <origin xyz="${-len_wagen_hinten/2-0.04} +0.006 ${height_wagen*2/3+0.0410}" rpy="${-camera_angle-1.57} 0 1.57"/>
+        <axis xyz="0 0 0"/>
+          <geometry>
+              <!-- <box size="${len_wagen_vorne} ${width_wagen} ${height_wagen}"/> -->
+              <mesh filename="package://floribot_simulation/meshes/Anschluss_Item_negativ.stl" scale="0.001 0.001 0.001" />
+          </geometry>
+          <material name="c">
+              <color rgba="0 0.9 0.9 1.0"/>
+          </material>
+      </visual>
+	  <inertial>
+		<mass value="0.1"/>
+        <inertia ixx="0.0" ixy="0.0" ixz="0.0" iyy="0.0" iyz="0.0" izz="0.0"/>
+      </inertial>
+  </link>
+  <joint name="jointCameraRearNegativ" type="fixed">
+       <parent link="CameraRearPositiv"/>
+       <child link="CameraRearNegativ"/>
+	   <origin xyz="0 0 0" rpy="0 0 0"/>
+  </joint>
   <!-- Laserscanner hinten -->
   <joint name="joint_rear_laser" type="fixed">
@@ -354,5 +442,5 @@
 		<mass value="2.4"/>
         <inertia ixx="0.013" ixy="0.0" ixz="0.0" iyy="0.023" iyz="0.0" izz="0.013"/>
-      </inertial>
+    </inertial>
   </link>
 <!-- Gelenk zwischen Hinterwagen und Rad HL -->
@@ -395,13 +483,4 @@
       <robotNamespace>floribot</robotNamespace>
     </plugin>
-    <!-- <plugin name="floribot_simulation" filename="libfloribot_simulation.so">
-    <activate_pid_control>yes</activate_pid_control>
-		<wheel_kp>1.0</wheel_kp>
-		<wheel_ki>0.5</wheel_ki>
-		<wheel_kd>0.01</wheel_kd>
-    </plugin> -->
   </gazebo>
-  <!--<xacro:sick_tim_5xx name="front_laser" ros_topic="laser_scanner_front"/>-->
-  <!-- <xacro:sick_tim_laser_gazebo_v0 name="laser" link="front_laser_mount_link" ros_topic="laser_scanner_front" update_rate="40" min_angle="-2.357" max_angle="2.357" min_range="0.05" max_range="4.0" samples="271"/> -->
-  <!-- <xacro:sick_tim_laser_gazebo_v0 name="laser" link="rear_laser_mount_link" ros_topic="laser_scanner_rear" update_rate="40" min_angle="-2.357" max_angle="2.357" min_range="0.05" max_range="4.0" samples="271"/> -->
 </robot>

Commit message: Laserscanner geändert So eingestellt, sodass er den Roboter nicht mehr ekennt

File: src/floribot_simulation/urdf/Floribot_final.urdf.xacro (robot description, xacro)
@@ -18,5 +18,5 @@
 <xacro:property name="y_joint_wheel_back" value="0.167" />
 <!-- Laserparameter -->
-<xacro:property name="x_laser_front" value="0.305" />
+<xacro:property name="x_laser_front" value="0.328" />
 <xacro:property name="x_laser_back" value="-0.33" />
 <xacro:property name="laser_height" value="0.03" />

File: src/sick_scan/urdf/sick_scan.urdf.xacro (robot description, xacro)
@@ -4,5 +4,5 @@
   xmlns:sensor="http://playerstage.sourceforge.net/gazebo/xmlschema/#sensor"
   xmlns:xacro="http://ros.org/wiki/xacro">
-  <xacro:macro name="sick_tim_5xx" params="name ros_topic min_angle:=-2.357 max_angle:=2.357 samples:=271">
+  <xacro:macro name="sick_tim_5xx" params="name ros_topic min_angle:=-2.00712864 max_angle:=2.00712864 samples:=697">
     <xacro:sick_tim name="${name}" ros_topic="${ros_topic}"
       length="0.06" width="0.06" height="0.079" mass="0.150" z_offset="0.05595"

Commit message: Effort-Problem

File: src/floribot_simulation/urdf/Floribot_final.urdf.xacro (robot description, xacro)
@@ -348,5 +348,5 @@
        <axis xyz="0 1 0"/>
        <origin xyz="${x_joint_wheel_front} ${y_joint_wheel_front} 0"/>
-        <limit effort="1.0" velocity="14.2857" />
+        <limit effort="100.0" velocity="14.2857" />
   </joint>
 <!-- Transmission -->
@@ -382,5 +382,5 @@
        <axis xyz="0 1 0"/>
        <origin xyz="${x_joint_wheel_front} -${y_joint_wheel_front} 0"/>
-       <limit effort="1.0" velocity="14.2857" />
+       <limit effort="100.0" velocity="14.2857" />
   </joint>
 <!-- Transmission -->
@@ -416,5 +416,5 @@
        <axis xyz="0 1 0"/>
        <origin xyz="${x_joint_wheel_back} -${y_joint_wheel_back} 0"/>
-       <limit effort="1.0" velocity="14.2857" />
+       <limit effort="100.0" velocity="14.2857" />
   </joint>
 <!-- Transmission -->
@@ -450,5 +450,5 @@
        <axis xyz="0 1 0"/>
        <origin xyz="${x_joint_wheel_back} ${y_joint_wheel_back} 0"/>
-       <limit effort="1.0" velocity="14.2857" />
+       <limit effort="100.0" velocity="14.2857" />
   </joint>
 <!-- Transmission -->

Commit message: Fixed inertia and mass

File: src/floribot_simulation/urdf/Floribot_final.urdf.xacro (robot description, xacro)
@@ -96,6 +96,6 @@
 	  <inertial>
     <origin xyz="0 0 ${wheel_radius}" rpy="0 0 0"/>
-		<mass value="33"/>
-        <inertia ixx="1.286541" ixy="0.0" ixz="0.0" iyy="0.457810" iyz="0.0" izz="1.063241"/>
+		<mass value="31"/>
+        <inertia ixx="0.3853" ixy="0.0001197" ixz="-0.0128" iyy="1.0" iyz="0.0000149" izz="0.8678"/>
       </inertial>
   </link>
@@ -284,5 +284,5 @@
     <origin xyz="0 0 ${wheel_radius}" rpy="0 0 0"/>
 		<mass value="33"/>
-        <inertia ixx="1.369982" ixy="0.0" ixz="0.0" iyy="0.487502" iyz="0.0" izz="1.132200"/>
+        <inertia ixx="0.4137" ixy="0.00027" ixz="0.007359" iyy="1.047" iyz="0.0001775" izz="0.9021"/>
       </inertial>
   </link>
@@ -373,5 +373,5 @@
 	  <inertial>
 		<mass value="2.4"/>
-        <inertia ixx="0.013" ixy="0.0" ixz="0.0" iyy="0.023" iyz="0.0" izz="0.013"/>
+        <inertia ixx="0.014" ixy="0.0" ixz="0.0" iyy="0.026" iyz="0.0" izz="0.014"/>
       </inertial>
   </link>
@@ -407,5 +407,5 @@
 	  <inertial>
 		<mass value="2.4"/>
-        <inertia ixx="0.013" ixy="0.0" ixz="0.0" iyy="0.023" iyz="0.0" izz="0.013"/>
+        <inertia ixx="0.014" ixy="0.0" ixz="0.0" iyy="0.026" iyz="0.0" izz="0.014"/>
       </inertial>
   </link>
@@ -441,5 +441,5 @@
 	  <inertial>
 		<mass value="2.4"/>
-        <inertia ixx="0.013" ixy="0.0" ixz="0.0" iyy="0.023" iyz="0.0" izz="0.013"/>
+        <inertia ixx="0.014" ixy="0.0" ixz="0.0" iyy="0.026" iyz="0.0" izz="0.014"/>
     </inertial>
   </link>
@@ -475,5 +475,5 @@
 	  <inertial>
 		<mass value="2.4"/>
-        <inertia ixx="0.013" ixy="0.0" ixz="0.0" iyy="0.023" iyz="0.0" izz="0.013"/>
+        <inertia ixx="0.014" ixy="0.0" ixz="0.0" iyy="0.026" iyz="0.0" izz="0.014"/>
       </inertial>
   </link>

Commit message: Scanner und Kamera vorne angepasst

File: src/floribot_simulation/urdf/Floribot_final.urdf.xacro (robot description, xacro)
@@ -18,12 +18,12 @@
 <xacro:property name="y_joint_wheel_back" value="0.167" />
 <!-- Laserparameter -->
-<xacro:property name="x_laser_front" value="0.328" />
+<xacro:property name="x_laser_front" value="0.332" />
 <xacro:property name="x_laser_back" value="-0.33" />
 <xacro:property name="laser_height" value="0.03" />
 <!-- Kameraparameter -->
-<xacro:property name="x_camera_front" value="0.3220" />
+<xacro:property name="x_camera_front" value="0.3133" />
 <xacro:property name="x_camera_back" value="-0.347" />
-<xacro:property name="camera_height" value="0.267" />
-<xacro:property name="camera_angle" value="0.26" />
+<xacro:property name="camera_height" value="0.263" />
+<xacro:property name="camera_angle" value="0.6" />
 <!--Verbindungsgelenkparameter (Skizze: |Vorderwagen|I==|Hinterwagen| -> I: Vertikaler Teil, ==: Horizontaler Teil) -->
 <xacro:property name="radius" value="0.008" />
@@ -109,5 +109,4 @@
         <axis xyz="0 0 0"/>
           <geometry>
-              <!-- <box size="${len_wagen_vorne} ${width_wagen} ${height_wagen}"/> -->
               <mesh filename="package://floribot_simulation/meshes/Anschluss_Item_positiv.stl" scale="0.001 0.001 0.001" />
           </geometry>
@@ -128,5 +127,5 @@
   <link name="CameraFrontNegativ">
       <visual>
-    	  <origin xyz="${len_wagen_vorne/2} -0.006 ${height_wagen*2/3+0.0410}" rpy="${-camera_angle-1.57} 0 -1.57"/>
+    	  <origin xyz="${len_wagen_vorne/2-0.0028} -0.006 ${height_wagen*2/3+0.0355}" rpy="${-camera_angle-1.57} 0 -1.57"/>
         <axis xyz="0 0 0"/>
           <geometry>
@@ -144,5 +143,5 @@
   </link>
   <joint name="jointCameraFrontNegativ" type="fixed">
-       <parent link="CameraFrontPositiv"/>
+      <parent link="CameraFrontPositiv"/>
        <child link="CameraFrontNegativ"/>
 	   <origin xyz="0 0 0" rpy="0 0 0"/>
@@ -150,9 +149,27 @@
   <!-- Laserscanner vorne -->
   <joint name="joint_front_laser" type="fixed">
-       <parent link="base_link"/>
-       <child link="front_laser_mount_link"/>
-	   <origin xyz="${x_laser_front} 0 ${laser_height}" rpy="3.14 0 0"/>
+    <parent link="base_link"/>
+    <child link="front_laser_mount_link"/>
+	  <origin xyz="${x_laser_front} 0 ${laser_height}" rpy="3.14 0 0"/>
   </joint>
   <xacro:sick_tim_5xx name="front_laser" ros_topic="laser_scanner_front"/>
+  <link name="laser_front_box">
+    <visual>
+      <origin xyz="0 0 0" rpy="0 0 0"/>
+      <axis xyz="0 0 0"/>
+        <geometry>
+            <box size="0.022 0.05 0.05"/> -->
+        </geometry>
+    </visual>
+	  <inertial>
+		  <mass value="0.1"/>
+      <inertia ixx="0.0" ixy="0.0" ixz="0.0" iyy="0.0" iyz="0.0" izz="0.0"/>
+    </inertial>
+  </link>
+  <joint name="joint_laser_box" type="fixed">
+     <parent link="base_link"/>
+     <child link="laser_front_box"/>
+     <origin xyz="${len_wagen_vorne/2-base2Vorderwagen+0.011} 0 -0.005" rpy="0 0 0"/>
+  </joint>
  <!-- Gelenk zwischen Vorderwagen und Verbindungsstueck -->
   <joint name="body_angle" type="revolute">

Commit message: Reifen eingefärbt

File: src/floribot_simulation/urdf/Floribot_final.urdf.xacro (robot description, xacro)
@@ -56,4 +56,9 @@
   </gazebo>
 </xacro:macro>
+<xacro:macro name = "wheelColor" params = "linkName">
+  <gazebo reference="${linkName}">
+    <material>Gazebo/Grey</material>
+  </gazebo>
+</xacro:macro>
   <!-- Base Link -->
   <link name="base_link">
@@ -495,4 +500,9 @@
       </inertial>
   </link>
+  <!-- Wheel Colors-->
+  <xacro:wheelColor linkName="frontLeft" />
+  <xacro:wheelColor linkName="frontRight" />
+  <xacro:wheelColor linkName="rearLeft" />
+  <xacro:wheelColor linkName="rearRight" />
 <!-- Gazebo plugin for ROS Control -->
   <gazebo>

Commit message: Roboter angemalt

File: src/floribot_simulation/urdf/Floribot_final.urdf.xacro (robot description, xacro)
@@ -58,5 +58,10 @@
 <xacro:macro name = "wheelColor" params = "linkName">
   <gazebo reference="${linkName}">
-    <material>Gazebo/Grey</material>
+    <material>Gazebo/FlatBlack</material>
+  </gazebo>
+</xacro:macro>
+<xacro:macro name= "darkGreyColor" params = "linkName">
+  <gazebo reference="${linkName}">
+    <material>Gazebo/DarkGrey</material>
   </gazebo>
 </xacro:macro>
@@ -105,4 +110,7 @@
       </inertial>
   </link>
+  <gazebo reference="Vorderwagen">
+      <material>Gazebo/Grey</material>
+  </gazebo>
   <!-- Kamera vorne-->
   <xacro:sensor_d435i name="front_camera" parent="base_link">
@@ -125,4 +133,5 @@
       </inertial>
   </link>
+  <xacro:darkGreyColor linkName = "CameraFrontPositiv" />
   <joint name="jointCameraFrontPositiv" type="fixed">
        <parent link="base_link"/>
@@ -147,4 +156,5 @@
       </inertial>
   </link>
+  <xacro:darkGreyColor linkName = "CameraFrontNegativ" />
   <joint name="jointCameraFrontNegativ" type="fixed">
       <parent link="CameraFrontPositiv"/>
@@ -172,4 +182,5 @@
     </inertial>
   </link>
+  <xacro:darkGreyColor linkName = "laser_front_box" />
   <joint name="joint_laser_box" type="fixed">
      <parent link="base_link"/>
@@ -217,4 +228,5 @@
       </inertial>
   </link>
+  <xacro:darkGreyColor linkName = "Gelenkteil_1" />
  <!-- Gelenk zwischen den beiden Verbindungsstuecken -->
   <joint name="Gelenk" type="revolute">
@@ -248,4 +260,5 @@
       </inertial>
   </link>
+  <xacro:darkGreyColor linkName = "Gelenkteil_2" />
  <!-- Gelenk zwischen Verbindungsstueck 2 und Hinterwagen -->
   <joint name="Gelenkteil_2_zu_Hinterwagen" type="fixed">
@@ -309,4 +322,7 @@
       </inertial>
   </link>
+  <gazebo reference="Hinterwagen">
+      <material>Gazebo/Grey</material>
+  </gazebo>
   <!-- Kamera hinten-->
   <xacro:sensor_d435i name="rear_camera" parent="Hinterwagen">
@@ -330,4 +346,5 @@
       </inertial>
   </link>
+  <xacro:darkGreyColor linkName = "CameraRearPositiv" />
   <joint name="jointCameraRearPositiv" type="fixed">
        <parent link="Hinterwagen"/>
@@ -352,4 +369,5 @@
       </inertial>
   </link>
+  <xacro:darkGreyColor linkName = "CameraRearNegativ" />
   <joint name="jointCameraRearNegativ" type="fixed">
        <parent link="CameraRearPositiv"/>

Commit message: Heckkamera angepasst

File: src/floribot_simulation/urdf/Floribot_final.urdf.xacro (robot description, xacro)
@@ -18,10 +18,10 @@
 <xacro:property name="y_joint_wheel_back" value="0.167" />
 <!-- Laserparameter -->
-<xacro:property name="x_laser_front" value="0.332" />
+<xacro:property name="x_laser_front" value="0.3315" />
 <xacro:property name="x_laser_back" value="-0.33" />
 <xacro:property name="laser_height" value="0.03" />
 <!-- Kameraparameter -->
 <xacro:property name="x_camera_front" value="0.3133" />
-<xacro:property name="x_camera_back" value="-0.347" />
+<xacro:property name="x_camera_back" value="-0.338" />
 <xacro:property name="camera_height" value="0.263" />
 <xacro:property name="camera_angle" value="0.6" />
@@ -354,5 +354,5 @@
   <link name="CameraRearNegativ">
       <visual>
-    	  <origin xyz="${-len_wagen_hinten/2-0.04} +0.006 ${height_wagen*2/3+0.0410}" rpy="${-camera_angle-1.57} 0 1.57"/>
+    	  <origin xyz="${-len_wagen_hinten/2-0.036} +0.006 ${height_wagen*2/3+0.0345}" rpy="${-camera_angle-1.57} 0 1.57"/>
         <axis xyz="0 0 0"/>
           <geometry>
