Commit message: clean up urdf

File: src/floribot_simulation/urdf/Floribot_final.urdf.xacro (robot description, xacro)
@@ -1,14 +1,14 @@
 <?xml version="1.0" encoding="UTF-8"?>
 <robot xmlns:xacro="http://www.ros.org/wiki/xacro" name="Floribot">
-<!-- Wagenparameter -->
-<xacro:property name="height_wagen" value="0.363" />
-<xacro:property name="width_wagen" value="0.213" />
-<xacro:property name="len_wagen_vorne" value="0.635" />
-<xacro:property name="len_wagen_hinten" value="0.605" />
-<!-- Ghost Elements -->
+<!-- wagon parameter -->
+<xacro:property name="height_wagon" value="0.363" />
+<xacro:property name="width_wagon" value="0.213" />
+<xacro:property name="length_wagon_front" value="0.635" />
+<xacro:property name="length_wagon_rear" value="0.605" />
+<!-- ghost elements -->
 <xacro:property name="ghost_size" value="0.01" />
-<xacro:property name="base2Vorderwagen" value="0.04" />
-<xacro:property name="Hinterwagenghost2Hinterwagen" value="0.025" />
-<!-- Reifenparameter -->
+<xacro:property name="base_2_front_wagon" value="0.04" />
+<xacro:property name="rear_wagon_ghost_2_rear_wagon" value="0.025" />
+<!-- wheel parameter -->
 <xacro:property name="wheel_radius" value="0.140" />
 <xacro:property name="wheel_thickness" value="0.09" />
@@ -17,35 +17,35 @@
 <xacro:property name="x_joint_wheel_back" value="0" />
 <xacro:property name="y_joint_wheel_back" value="0.167" />
-<!-- Laserparameter -->
+<!-- laser parameter -->
 <xacro:property name="x_laser_front" value="0.3315" />
 <xacro:property name="x_laser_back" value="-0.33" />
 <xacro:property name="laser_height" value="0.03" />
-<!-- Kameraparameter -->
+<!-- camera parameter -->
 <xacro:property name="x_camera_front" value="0.3133" />
 <xacro:property name="x_camera_back" value="-0.338" />
 <xacro:property name="camera_height" value="0.263" />
 <xacro:property name="camera_angle" value="0.6" />
-<!--Verbindungsgelenkparameter (Skizze: |Vorderwagen|I==|Hinterwagen| -> I: Vertikaler Teil, ==: Horizontaler Teil) -->
+<!--articulated joint parameter -->
 <xacro:property name="radius" value="0.008" />
-<xacro:property name="vertikal_length" value="0.06" />
+<xacro:property name="vertical_length" value="0.06" />
 <xacro:property name="horizontal_length" value="0.055" />
-<xacro:property name="WheelJoint2MidJoint" value="0.383" />
-<xacro:property name="JointHeight" value="0.015" />
-<!-- Hinzufuegen des Laserscanners -->
+<xacro:property name="wheel_joint_2_mid_joint" value="0.383" />
+<xacro:property name="joint_height" value="0.015" />
+<!-- add laserscanners -->
 <xacro:include filename="$(find sick_scan)/urdf/sick_scan.urdf.xacro" />
 <xacro:include filename="$(find realsense2_description)/urdf/_d435i.urdf.xacro" />
-<!-- Makro fuer Wheel Tranmission -->
-<xacro:macro name="wheelTransGaz" params="position">
+<!-- macro wheel tranmission -->
+<xacro:macro name="wheel_transmission" params="position">
   <transmission name="joint_${position}_trans">
-        <type>transmission_interface/SimpleTransmission</type>
-        <joint name="joint_${position}">
-          <hardwareInterface>hardware_interface/VelocityJointInterface</hardwareInterface>
-        </joint>
-        <actuator name="joint_${position}_motor">
-          <hardwareInterface>hardware_interface/VelocityActuatorInterface</hardwareInterface>
-          <mechanicalReduction>1</mechanicalReduction>
-        </actuator>
+    <type>transmission_interface/SimpleTransmission</type>
+    <joint name="joint_${position}">
+      <hardwareInterface>hardware_interface/VelocityJointInterface</hardwareInterface>
+    </joint>
+    <actuator name="joint_${position}_motor">
+      <hardwareInterface>hardware_interface/VelocityActuatorInterface</hardwareInterface>
+      <mechanicalReduction>1</mechanicalReduction>
+    </actuator>
   </transmission>
-  <!-- hardware_interface/VelocityJointInterface -->
+  <!-- friction and damping coefficents for gazebo simulation -->
   <gazebo reference="${position}">
     <mu1 value="0.5"/>
@@ -56,9 +56,11 @@
   </gazebo>
 </xacro:macro>
-<xacro:macro name = "wheelColor" params = "linkName">
+<!-- macro wheel color for gazbeo -->
+<xacro:macro name = "wheel_color" params = "linkName">
   <gazebo reference="${linkName}">
     <material>Gazebo/FlatBlack</material>
   </gazebo>
 </xacro:macro>
+<!-- macro grey color for gazbeo -->
 <xacro:macro name= "darkGreyColor" params = "linkName">
   <gazebo reference="${linkName}">
@@ -66,466 +68,479 @@
   </gazebo>
 </xacro:macro>
-  <!-- Base Link -->
-  <link name="base_link">
-      <visual>
-    	  <origin xyz="0 0 ${wheel_radius + ghost_size}" rpy="0 0 0"/>
-        <axis xyz="0 0 0"/>
-          <geometry>
-              <box size="${ghost_size} ${ghost_size} ${ghost_size}"/>
-          </geometry>
-          <material name="c">
-              <color rgba="0 0.9 0.9 1.0"/>
-          </material>
-      </visual>
-  </link>
-   <!-- Gelenk zwischen Vorderwagen und base_link -->
-  <joint name="base_zu_Vorderwagen" type="fixed">
-       <parent link="base_link"/>
-       <child link="Vorderwagen"/>
-	   <origin xyz="${-base2Vorderwagen} 0 0"/>
+<!-- base link -->
+<link name="base_link">
+  <visual>
+    <origin xyz="0 0 ${wheel_radius + ghost_size}" rpy="0 0 0"/>
+    <axis xyz="0 0 0"/>
+    <geometry>
+        <box size="${ghost_size} ${ghost_size} ${ghost_size}"/>
+    </geometry>
+    <material name="c">
+        <color rgba="0 0.9 0.9 1.0"/>
+    </material>
+  </visual>
+</link>
+  <!-- joint between front wagon and base_link -->
+<joint name="j_base_2_front_wagon" type="fixed">
+  <parent link="base_link"/>
+  <child link="front_wagon"/>
+  <origin xyz="${-base_2_front_wagon} 0 0"/>
+</joint>
+<!-- front wagon -->
+<link name="front_wagon">
+  <visual>
+    <origin xyz="-${length_wagon_front/2+0.0255} 0 -${wheel_radius}" rpy="0 0 0"/>
+    <axis xyz="0 0 0"/>
+    <geometry>
+      <mesh filename="package://floribot_simulation/meshes/Vorderwagen.stl" scale="0.001 0.001 0.001" />
+    </geometry>
+    <material name="c">
+      <color rgba="0 0.9 0.9 1.0"/>
+    </material>
+  </visual>
+  <collision>
+    <origin xyz="0 0 ${wheel_radius}" rpy="0 0 0"/>
+    <geometry>
+      <box size="${length_wagon_front} ${width_wagon} ${height_wagon}"/>
+    </geometry>
+  </collision>
+  <inertial>
+    <origin xyz="0 0 ${wheel_radius}" rpy="0 0 0"/>
+    <mass value="31"/>
+    <inertia ixx="0.3853" ixy="0.0001197" ixz="-0.0128" iyy="1.0" iyz="0.0000149" izz="0.8678"/>
+  </inertial>
+</link>
+<!-- gazebo color front wagon -->
+<gazebo reference="front_wagon">
+  <material>Gazebo/Grey</material>
+</gazebo>
+<!-- front camera -->
+<xacro:sensor_d435i name="front_camera" parent="base_link">
+  <origin xyz="${x_camera_front} 0 ${camera_height}" rpy="0 ${camera_angle} 0"/>
+</xacro:sensor_d435i>
+<!-- front camera positiv link -->
+<link name="camera_front_positiv">
+  <visual>
+    <origin xyz="${length_wagon_front/2-0.06} -0.0225 ${height_wagon*2/3+0.033}" rpy="0 1.57 0"/>
+    <axis xyz="0 0 0"/>
+    <geometry>
+      <mesh filename="package://floribot_simulation/meshes/Anschluss_Item_positiv.stl" scale="0.001 0.001 0.001" />
+    </geometry>
+    <material name="c">
+      <color rgba="0 0.9 0.9 1.0"/>
+    </material>
+  </visual>
+  <inertial>
+    <mass value="0.1"/>
+    <inertia ixx="0.0" ixy="0.0" ixz="0.0" iyy="0.0" iyz="0.0" izz="0.0"/>
+  </inertial>
+</link>
+<!-- gazebo camera link color -->
+<xacro:darkGreyColor linkName = "camera_front_positiv" />
+<!-- joint between camera front positiv and base link -->
+<joint name="j_camera_front_positiv" type="fixed">
+  <parent link="base_link"/>
+  <child link="camera_front_positiv"/>
+  <origin xyz="0 0 0" rpy="0 0 0"/>
+</joint>
+<!-- front camera negativ link -->
+<link name="camera_front_negativ">
+  <visual>
+   <origin xyz="${length_wagon_front/2-0.0028} -0.006 ${height_wagon*2/3+0.0355}" rpy="${-camera_angle-1.57} 0 -1.57"/>
+    <axis xyz="0 0 0"/>
+    <geometry>
+      <mesh filename="package://floribot_simulation/meshes/Anschluss_Item_negativ.stl" scale="0.001 0.001 0.001" />
+    </geometry>
+    <material name="c">
+      <color rgba="0 0.9 0.9 1.0"/>
+    </material>
+  </visual>
+  <inertial>
+    <mass value="0.1"/>
+    <inertia ixx="0.0" ixy="0.0" ixz="0.0" iyy="0.0" iyz="0.0" izz="0.0"/>
+  </inertial>
+</link>
+<!-- gazebo camera link color -->
+<xacro:darkGreyColor linkName = "camera_front_negativ" />
+<!-- joint between camera front positiv and negativ -->
+<joint name="j_camera_front_negativ" type="fixed">
+  <parent link="camera_front_positiv"/>
+  <child link="camera_front_negativ"/>
+  <origin xyz="0 0 0" rpy="0 0 0"/>
+</joint>
+<!-- joint laserscanner front  -->
+<joint name="joint_front_laser" type="fixed">
+  <parent link="base_link"/>
+  <child link="front_laser_mount_link"/>
+  <origin xyz="${x_laser_front} 0 ${laser_height}" rpy="3.14 0 0"/>
+</joint>
+<!-- link laserscanner front -->
+<xacro:sick_tim_5xx name="front_laser" ros_topic="laser_scanner_front"/>
+<!-- distance box laserscanner front -->
+<link name="laser_front_box">
+  <visual>
+    <origin xyz="0 0 0" rpy="0 0 0"/>
+    <axis xyz="0 0 0"/>
+    <geometry>
+      <box size="0.022 0.05 0.05"/> -->
+    </geometry>
+  </visual>
+  <inertial>
+    <mass value="0.1"/>
+    <inertia ixx="0.0" ixy="0.0" ixz="0.0" iyy="0.0" iyz="0.0" izz="0.0"/>
+  </inertial>
+</link>
+<!-- gazebo color scanner box -->
+<xacro:darkGreyColor linkName = "laser_front_box" />
+<!-- joint between laserscanner box and base link-->
+<joint name="j_laser_box" type="fixed">
+    <parent link="base_link"/>
+    <child link="laser_front_box"/>
+    <origin xyz="${length_wagon_front/2-base_2_front_wagon+0.011} 0 -0.005" rpy="0 0 0"/>
+</joint>
+<!-- joint between base link and first part of the articulated joint (body_angle) -->
+<joint name="body_angle" type="revolute">
+    <axis xyz="0 0 1"/>
+    <limit effort="1.0" lower="-1.57" upper="1.57" velocity="0.5"/>
+    <parent link="base_link"/>
+    <child link="connection_part_1"/>
+    <origin xyz="${-wheel_joint_2_mid_joint} 0 -${joint_height}"/>
+</joint>
+<!-- transmisson for body angle -> this is required to present this joint in floribot/joint_states -->
+<transmission name="body_angle_trans">
+  <type>transmission_interface/SimpleTransmission</type>
+  <joint name="body_angle">
+    <hardwareInterface>hardware_interface/VelocityJointInterface</hardwareInterface>
   </joint>
-  <!-- Vorderwagen -->
-  <link name="Vorderwagen">
-      <visual>
-    	  <origin xyz="-${len_wagen_vorne/2+0.0255} 0 -${wheel_radius}" rpy="0 0 0"/>
-        <axis xyz="0 0 0"/>
-          <geometry>
-              <!-- <box size="${len_wagen_vorne} ${width_wagen} ${height_wagen}"/> -->
-              <mesh filename="package://floribot_simulation/meshes/Vorderwagen.stl" scale="0.001 0.001 0.001" />
-          </geometry>
-          <material name="c">
-              <color rgba="0 0.9 0.9 1.0"/>
-          </material>
-      </visual>
-      <collision>
-        <origin xyz="0 0 ${wheel_radius}" rpy="0 0 0"/>
-		    <geometry>
-              <box size="${len_wagen_vorne} ${width_wagen} ${height_wagen}"/>
-            </geometry>
-	  </collision>
-	  <inertial>
-    <origin xyz="0 0 ${wheel_radius}" rpy="0 0 0"/>
-		<mass value="31"/>
-        <inertia ixx="0.3853" ixy="0.0001197" ixz="-0.0128" iyy="1.0" iyz="0.0000149" izz="0.8678"/>
-      </inertial>
-  </link>
-  <gazebo reference="Vorderwagen">
-      <material>Gazebo/Grey</material>
-  </gazebo>
-  <!-- Kamera vorne-->
-  <xacro:sensor_d435i name="front_camera" parent="base_link">
-    <origin xyz="${x_camera_front} 0 ${camera_height}" rpy="0 ${camera_angle} 0"/>
-  </xacro:sensor_d435i>
-  <link name="CameraFrontPositiv">
-      <visual>
-    	  <origin xyz="${len_wagen_vorne/2-0.06} -0.0225 ${height_wagen*2/3+0.033}" rpy="0 1.57 0"/>
-        <axis xyz="0 0 0"/>
-          <geometry>
-              <mesh filename="package://floribot_simulation/meshes/Anschluss_Item_positiv.stl" scale="0.001 0.001 0.001" />
-          </geometry>
-          <material name="c">
-              <color rgba="0 0.9 0.9 1.0"/>
-          </material>
-      </visual>
-	  <inertial>
-		<mass value="0.1"/>
-        <inertia ixx="0.0" ixy="0.0" ixz="0.0" iyy="0.0" iyz="0.0" izz="0.0"/>
-      </inertial>
-  </link>
-  <xacro:darkGreyColor linkName = "CameraFrontPositiv" />
-  <joint name="jointCameraFrontPositiv" type="fixed">
-       <parent link="base_link"/>
-       <child link="CameraFrontPositiv"/>
-	   <origin xyz="0 0 0" rpy="0 0 0"/>
-  </joint>
-  <link name="CameraFrontNegativ">
-      <visual>
-    	  <origin xyz="${len_wagen_vorne/2-0.0028} -0.006 ${height_wagen*2/3+0.0355}" rpy="${-camera_angle-1.57} 0 -1.57"/>
-        <axis xyz="0 0 0"/>
-          <geometry>
-              <!-- <box size="${len_wagen_vorne} ${width_wagen} ${height_wagen}"/> -->
-              <mesh filename="package://floribot_simulation/meshes/Anschluss_Item_negativ.stl" scale="0.001 0.001 0.001" />
-          </geometry>
-          <material name="c">
-              <color rgba="0 0.9 0.9 1.0"/>
-          </material>
-      </visual>
-	  <inertial>
-		<mass value="0.1"/>
-        <inertia ixx="0.0" ixy="0.0" ixz="0.0" iyy="0.0" iyz="0.0" izz="0.0"/>
-      </inertial>
-  </link>
-  <xacro:darkGreyColor linkName = "CameraFrontNegativ" />
-  <joint name="jointCameraFrontNegativ" type="fixed">
-      <parent link="CameraFrontPositiv"/>
-       <child link="CameraFrontNegativ"/>
-	   <origin xyz="0 0 0" rpy="0 0 0"/>
-  </joint>
-  <!-- Laserscanner vorne -->
-  <joint name="joint_front_laser" type="fixed">
-    <parent link="base_link"/>
-    <child link="front_laser_mount_link"/>
-	  <origin xyz="${x_laser_front} 0 ${laser_height}" rpy="3.14 0 0"/>
-  </joint>
-  <xacro:sick_tim_5xx name="front_laser" ros_topic="laser_scanner_front"/>
-  <link name="laser_front_box">
-    <visual>
-      <origin xyz="0 0 0" rpy="0 0 0"/>
-      <axis xyz="0 0 0"/>
-        <geometry>
-            <box size="0.022 0.05 0.05"/> -->
-        </geometry>
-    </visual>
-	  <inertial>
-		  <mass value="0.1"/>
-      <inertia ixx="0.0" ixy="0.0" ixz="0.0" iyy="0.0" iyz="0.0" izz="0.0"/>
+  <actuator name="body_angle_motor">
+    <mechanicalReduction>1</mechanicalReduction>
+  </actuator>
+</transmission>
+<!-- connection part 1 of the articulated joint (vertical one) -->
+<link name="connection_part_1">
+  <visual>
+    <origin xyz="0 0 0" rpy="0 0 0"/>
+    <axis xyz="0 0 0"/>
+    <geometry>
+      <cylinder length="${vertical_length}" radius="${radius}"/>
+    </geometry>
+    <material name="r">
+      <color rgba="0.9 0 0 1.0"/>
+    </material>
+  </visual>
+  <collision>
+    <origin xyz="0 0 0" rpy="0 0 0"/>
+    <geometry>
+      <cylinder length="${vertical_length}" radius="${radius}"/>
+    </geometry>
+  </collision>
+  <inertial>
+    <mass value="0.01"/>
+    <inertia ixx="0.000004" ixy="0.0" ixz="0.0" iyy="0.0" iyz="0.0" izz="0.000004"/>
+  </inertial>
+</link>
+<!-- gazebo color -->
+<xacro:darkGreyColor linkName = "connection_part_1" />
+<!-- revolute joint between both connection parts for the articulated joint -->
+<joint name="j_revolute_front_rear" type="revolute">
+  <axis xyz="1 0 0"/>
+  <limit effort="1.0" lower="-1.57" upper="1.57" velocity="0.5"/>-
+  <parent link="connection_part_1"/>
+  <child link="connection_part_2"/>
+  <origin xyz="${-horizontal_length/2 - radius} 0 0"/>
+</joint>
+<!-- connection part 2 -->
+<link name="connection_part_2">
+  <visual>
+    <origin xyz="0 0 0" rpy="0 1.57 0"/>
+    <axis xyz="0 0 0.025"/>
+    <geometry>
+      <cylinder length="${horizontal_length}" radius="${radius}"/>
+    </geometry>
+    <material name="r">
+      <color rgba="0.9 0 0 1.0"/>
+    </material>
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